File: Kicad/Voldy_Life_Support/Voldy_Life_Support.kicad_pcb (KiCad board)
At the start: 2 copper layers, 23 parts, among them U4 ESP32_Lolin, U555 NE555P

Commit message: Add SHT20, SCD40
Parts:
- added REF**: , Resistor_THT:R_Axial_DIN0207_L6.3mm_D2.5mm_P7.62mm_Horizontal, F.Cu at (157.5, 116.8)
- added REF**: SIP-4, ESP32:SIP-4, F.Cu at (158.8, 92.7)
- added REF**: SIP-2, ESP32:SIP-2, F.Cu at (188.0, 123.2)
- added REF**: SIP-2, ESP32:SIP-2, F.Cu at (180.3, 123.2)
- added UBTN1: 2-Pin, ESP32:SIP-2, F.Cu at (171.4, 110.5)
- added UBTN1: 2-Pin, ESP32:SIP-2, F.Cu at (163.8, 110.5)
Routing:
- net (no net): track 0.00 -> 179.5 mm, vias 0 -> 1
- net +3V3: track 119.4 -> 178.0 mm, vias 2 -> 5
- net Net-(U4-Pad4): track 17.8 -> 43.1 mm
- net Net-(U4-Pad2): track 25.4 -> 45.7 mm, vias 0 -> 1
- net GND: track 249.0 -> 266.8 mm
